File: bitaxeMax4.kicad_sch (KiCad schematic)
At the start: 90 parts, among them IC1 BM1397_mode1, J1 Conn_01x01, J2 Conn_01x01, J3 Conn_01x05, J4 Conn_01x02, J5 Conn_01x03, U1 SN74LVC1T45QDCKRQ1, U2 oscillator, U3 SN74LVC1T45QDCKRQ1, U4 SN74LVC1T45QDCKRQ1, U5 MCP1824, U6 MCP1824, U7 ESP32-C3-DEVKITC-02, U8 NCT218

Commit message: schematic progress. still not done
Parts:
- removed R6: 10k, DayMiner:R0402, symbol Device:R_US
- added C? (x36): 587-5514-1-ND, DayMiner:C0402, symbol DayMiner-eagle-import:CAP0402
- added IC? (x2): BM1397_mode0, symbol bitaxe:BM1397_mode0
- added IC?: BM1397_mode1, DayMiner:SON45P800X800X70-33T645X800N, symbol bitaxe:BM1397_mode1
- added JP? (x6): SolderJumper_2_Open, Jumper:SolderJumper-2_P1.3mm_Open_RoundedPad1.0x1.5mm, symbol Jumper:SolderJumper_2_Open
- added JP? (x3): SolderJumper_2_Bridged, Jumper:SolderJumper-2_P1.3mm_Bridged2Bar_RoundedPad1.0x1.5mm, symbol Jumper:SolderJumper_2_Bridged
- added TP? (x3): TestPoint, TestPoint:TestPoint_Pad_D1.5mm, symbol Connector:TestPoint
Connections:
- net 0V8: now also C?.1, C?.1, C?.1, C?.1, C?.1, C?.1, IC?.14 (PLL_VDD), IC?.14 (PLL_VDD), IC?.14 (PLL_VDD), IC?.15 (VDDIO_08_0), IC?.15 (VDDIO_08_0), IC?.15 (VDDIO_08_0), IC?.18 (VDDIO_08_1), IC?.18 (VDDIO_08_1), IC?.18 (VDDIO_08_1)
- net 1V8: now also C?.1, C?.1, C?.1, C?.1, C?.1, C?.1, IC?.16 (VDDIO_18_0), IC?.16 (VDDIO_18_0), IC?.16 (VDDIO_18_0), IC?.17 (VDDIO_18_1), IC?.17 (VDDIO_18_1), IC?.17 (VDDIO_18_1)
- net GND: now also C?.1, C?.1, C?.1, C?.2, C?.2, C?.2, C?.2, C?.2, C?.2, C?.2, C?.2, C?.2, C?.2, C?.2, C?.2, C?.2, C?.2, C?.2, IC?.13 (PLL_VSS), IC?.13 (PLL_VSS), IC?.13 (PLL_VSS), IC?.19 (VSS), IC?.19 (VSS), IC?.19 (VSS), IC?.20 (PIN_MODE), IC?.20 (PIN_MODE), IC?.20 (PIN_MODE), IC?.34 (VSS_0), IC?.34 (VSS_0), IC?.34 (VSS_0), JP?.1 (A), JP?.1 (A), JP?.1 (A), JP?.1 (A), JP?.1 (A), JP?.1 (A), JP?.1 (A), JP?.1 (A), JP?.1 (A), TP?.1, TP?.1, TP?.1
- net VDD: now also C?.1, C?.1, C?.1, C?.2, C?.2, C?.2, IC?.33 (VDD), IC?.33 (VDD), IC?.33 (VDD)
- net at IC1.26 (CO), TP5.1: now also IC?.28 (CI)
- net at IC1.25 (CLKO), TP6.1: now also IC?.29 (CLKI)
- net at IC1.27 (RI): now also IC?.27 (RO)
- net at IC1.28 (NRSTO), TP4.1: now also IC?.26 (NRSTI)
- net at IC1.29 (BO), TP3.1: now also IC?.25 (BI)
- new net: C?.1, C?.2, IC?.3 (VDD1_0) (x3)
- new net: C?.1, C?.2, IC?.2 (VDD2_0) (x3)
- new net: C?.1, C?.2, IC?.1 (VDD3_0) (x3)
- new net: C?.1, C?.2, IC?.30 (VDD1_1) (x3)
- new net: IC?.25 (BI), IC?.29 (BO)
- new net: IC?.26 (NRSTI), IC?.28 (NRSTO)
- new net: IC?.27 (RI), IC?.27 (RO)
- new net: IC?.26 (CO), IC?.28 (CI)
- new net: IC?.25 (CLKO), IC?.29 (CLKI)
- new net: C?.1, C?.2, IC?.31 (VDD2_1) (x3)
- new net: C?.1, C?.2, IC?.32 (VDD3_1) (x3)
- new net: IC?.4 (ADDR0), JP?.2 (B) (x3)
- new net: IC?.5 (ADDR1), JP?.2 (B) (x3)
- new net: IC?.6 (ADDR2), JP?.2 (B) (x3)
- new net: IC?.10 (RI), IC?.10 (RO)
- new net: IC?.11 (CI), IC?.9 (CO)
- new net: IC?.12 (CLKI), IC?.8 (CLKO)
- new net: IC?.12 (BO), IC?.8 (BI)
- new net: IC?.11 (NRSTO), IC?.9 (NRSTI)
Other:
- note added: "bitaxeMAX4"
- note removed: "bitaxeMAX"
- title: le bitaxe -> le bitaxeMax4
- moved on the sheet: C1, C10, C11, C12, C13, C14, C15, C16, C17, C18, C2, C3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
